File: PCB/Cape/agricoltura-madre-cape/RS485_Interface.sch (KiCad schematic (older format))
At the start: 14 parts

Commit message: Datasheets and BBG version
Finished initial schematic for BBG Gateway version and added datasheets for ST sub 1GHZ RF hardware.
Parts:
- gave numbers to parts that had none: 14
Changed lines of the file:
@@
 RS485_UART_RX1
 $Comp
-L power:GND #PWR?
+L power:GND #PWR027
 U 1 1 5F0382D4
 P 4850 6350
-F 0 "#PWR?" H 4850 6100 50  0001 C CNN
+F 0 "#PWR027" H 4850 6100 50  0001 C CNN
 F 1 "GND" H 4855 6177 50  0000 C CNN
 F 2 "" H 4850 6350 50  0001 C CNN
@@
 RS485_UART_RX2
 $Comp
-L power:+3V3 #PWR?
+L power:+3V3 #PWR016
 U 1 1 5F01A2C3
 P 2900 3050
-F 0 "#PWR?" H 2900 2900 50  0001 C CNN
+F 0 "#PWR016" H 2900 2900 50  0001 C CNN
 F 1 "+3V3" H 2915 3223 50  0000 C CNN
 F 2 "" H 2900 3050 50  0001 C CNN
@@
 $EndComp
 $Comp
-L AVR-KiCAD-Lib-Capacitors:C0402C104K9PACTU C?
+L AVR-KiCAD-Lib-Capacitors:C0402C104K9PACTU C1
 U 1 1 5F01065A
 P 3350 3250
-F 0 "C?" V 3329 3378 50  0000 L CNN
+F 0 "C1" V 3329 3378 50  0000 L CNN
 F 1 "C0402C104K9PACTU" H 3400 3450 50  0001 C CNN
 F 2 "AVR-KiCAD-Lib-Resistors:R0402" H 3150 3250 50  0001 C CNN
@@
 $EndComp
 $Comp
-L AVR-KiCAD-Lib-Connectors:0395121004 T?
+L AVR-KiCAD-Lib-Connectors:0395121004 T1
 U 1 1 5F06639C
 P 10200 2350
-F 0 "T?" H 10200 2500 50  0000 L CNN
+F 0 "T1" H 10200 2500 50  0000 L CNN
 F 1 "0395121004" H 10200 1900 50  0000 L CNN
 F 2 "AVR-KiCAD-Lib-Connectors:0395121004" H 9250 3400 50  0001 C CNN
@@
 	9250 2350 9250 2450
 $Comp
-L AVR-KiCAD-Lib-ICs:MAX13450EAUD+ U?
+L AVR-KiCAD-Lib-ICs:MAX13450EAUD+ U1
 U 1 1 5EF47AA2
 P 5150 1550
-F 0 "U?" H 5200 1600 50  0000 C CNN
+F 0 "U1" H 5200 1600 50  0000 C CNN
 F 1 "MAX13450EAUD+" H 5200 1650 50  0001 C CNN
 F 2 "AVR-KiCAD-Lib-ICs:MAX13450EAUD&plus_" H 4650 2200 50  0001 C CNN
@@
 	6150 2450 9250 2450
 $Comp
-L AVR-KiCAD-Lib-ICs:MAX13450EAUD+ U?
+L AVR-KiCAD-Lib-ICs:MAX13450EAUD+ U2
 U 1 1 5EF6EA13
 P 5150 4750
-F 0 "U?" H 5200 4800 50  0000 C CNN
+F 0 "U2" H 5200 4800 50  0000 C CNN
 F 1 "MAX13450EAUD+" H 5200 4850 50  0001 C CNN
 F 2 "AVR-KiCAD-Lib-ICs:MAX13450EAUD&plus_" H 4650 5400 50  0001 C CNN
@@
 $EndComp
 $Comp
-L power:GND #PWR?
+L power:GND #PWR025
 U 1 1 5EF78348
 P 4850 3150
-F 0 "#PWR?" H 4850 2900 50  0001 C CNN
+F 0 "#PWR025" H 4850 2900 50  0001 C CNN
 F 1 "GND" H 4855 2977 50  0000 C CNN
 F 2 "" H 4850 3150 50  0001 C CNN
@@
 	4850 6250 4850 6350
 $Comp
-L power:+5V #PWR?
+L power:+5V #PWR022
 U 1 1 5EF7B017
 P 4150 6150
-F 0 "#PWR?" H 4150 6000 50  0001 C CNN
+F 0 "#PWR022" H 4150 6000 50  0001 C CNN
 F 1 "+5V" H 4165 6323 50  0000 C CNN
 F 2 "" H 4150 6150 50  0001 C CNN
@@
 $EndComp
 $Comp
-L power:GND #PWR?
+L power:GND #PWR019
 U 1 1 5F0382C0
 P 3400 6600
-F 0 "#PWR?" H 3400 6350 50  0001 C CNN
+F 0 "#PWR019" H 3400 6350 50  0001 C CNN
 F 1 "GND" H 3405 6427 50  0000 C CNN
 F 2 "" H 3400 6600 50  0001 C CNN
@@
 $EndComp
 $Comp
-L AVR-KiCAD-Lib-Capacitors:C0402C104K9PACTU C?
+L AVR-KiCAD-Lib-Capacitors:C0402C104K9PACTU C2
 U 1 1 5F03829B
 P 3400 6350
-F 0 "C?" V 3379 6478 50  0000 L CNN
+F 0 "C2" V 3379 6478 50  0000 L CNN
 F 1 "C0402C104K9PACTU" H 3450 6550 50  0001 C CNN
 F 2 "AVR-KiCAD-Lib-Resistors:R0402" H 3200 6350 50  0001 C CNN
@@
 $EndComp
 $Comp
-L AVR-KiCAD-Lib-Capacitors:CGA3E2X7R1H104K080AA C?
+L AVR-KiCAD-Lib-Capacitors:CGA3E2X7R1H104K080AA C4
 U 1 1 5EF8977D
 P 4150 6350
-F 0 "C?" V 4129 6478 50  0000 L CNN
+F 0 "C4" V 4129 6478 50  0000 L CNN
 F 1 "CGA3E2X7R1H104K080AA" H 4200 6550 50  0001 C CNN
 F 2 "AVR-KiCAD-Lib-Capacitors:C0603" H 3950 6350 50  0001 C CNN
@@
 	4700 5750 4700 6150
 $Comp
-L power:GND #PWR?
+L power:GND #PWR023
 U 1 1 5EFA0EF6
 P 4150 6600
-F 0 "#PWR?" H 4150 6350 50  0001 C CNN
+F 0 "#PWR023" H 4150 6350 50  0001 C CNN
 F 1 "GND" H 4155 6427 50  0000 C CNN
 F 2 "" H 4150 6600 50  0001 C CNN
@@
 $EndComp
 $Comp
-L power:+5V #PWR?
+L power:+5V #PWR020
 U 1 1 5EFA9F3D
 P 4150 3050
-F 0 "#PWR?" H 4150 2900 50  0001 C CNN
+F 0 "#PWR020" H 4150 2900 50  0001 C CNN
 F 1 "+5V" H 4165 3223 50  0000 C CNN
 F 2 "" H 4150 3050 50  0001 C CNN
@@
 $EndComp
 $Comp
-L AVR-KiCAD-Lib-Capacitors:CGA3E2X7R1H104K080AA C?
+L AVR-KiCAD-Lib-Capacitors:CGA3E2X7R1H104K080AA C3
 U 1 1 5EFA9F5C
 P 4150 3250
-F 0 "C?" V 4129 3378 50  0000 L CNN
+F 0 "C3" V 4129 3378 50  0000 L CNN
 F 1 "CGA3E2X7R1H104K080AA" H 4200 3450 50  0001 C CNN
 F 2 "AVR-KiCAD-Lib-Capacitors:C0603" H 3950 3250 50  0001 C CNN
@@
 	4700 2550 4700 3050
 $Comp
-L power:GND #PWR?
+L power:GND #PWR021
 U 1 1 5EFA9F88
 P 4150 3500
-F 0 "#PWR?" H 4150 3250 50  0001 C CNN
+F 0 "#PWR021" H 4150 3250 50  0001 C CNN
 F 1 "GND" H 4155 3327 50  0000 C CNN
 F 2 "" H 4150 3500 50  0001 C CNN
@@
 	9200 5350 10000 5350
 $Comp
-L AVR-KiCAD-Lib-Connectors:0395121004 T?
+L AVR-KiCAD-Lib-Connectors:0395121004 T2
 U 1 1 5F0711FA
 P 10200 5550
-F 0 "T?" H 10200 5700 50  0000 L CNN
+F 0 "T2" H 10200 5700 50  0000 L CNN
 F 1 "0395121004" H 10200 5100 50  0000 L CNN
 F 2 "AVR-KiCAD-Lib-Connectors:0395121004" H 9250 6600 50  0001 C CNN
@@
 	6150 5650 9300 5650
 $Comp
-L AVR-KiCAD-Lib-Resistors:RC0402FR-071KL R?
+L AVR-KiCAD-Lib-Resistors:RC0402FR-071KL R11
 U 1 1 5EFF327C
 P 4850 4550
-F 0 "R?" V 4804 4637 50  0000 L CNN
+F 0 "R11" V 4804 4637 50  0000 L CNN
 F 1 "RC0402FR-071KL" V 4850 4638 50  0001 L CNN
 F 2 "AVR-KiCAD-Lib-Resistors:R0402" H 4850 4550 50  0001 C CNN
@@
 Connection ~ 4850 4850
 $Comp
-L AVR-KiCAD-Lib-Resistors:RC0402FR-071KL R?
+L AVR-KiCAD-Lib-Resistors:RC0402FR-071KL R10
 U 1 1 5EFFB143
 P 4850 1350
-F 0 "R?" V 4804 1437 50  0000 L CNN
+F 0 "R10" V 4804 1437 50  0000 L CNN
 F 1 "RC0402FR-071KL" V 4850 1438 50  0001 L CNN
 F 2 "AVR-KiCAD-Lib-Resistors:R0402" H 4850 1350 50  0001 C CNN
@@
 Connection ~ 4850 1650
 $Comp
-L power:+3V3 #PWR?
+L power:+3V3 #PWR024
 U 1 1 5F001021
 P 4850 1150
-F 0 "#PWR?" H 4850 1000 50  0001 C CNN
+F 0 "#PWR024" H 4850 1000 50  0001 C CNN
 F 1 "+3V3" H 4865 1323 50  0000 C CNN
 F 2 "" H 4850 1150 50  0001 C CNN
@@
 $EndComp
 $Comp
-L power:+3V3 #PWR?
+L power:+3V3 #PWR026
 U 1 1 5F0017EA
 P 4850 4350
-F 0 "#PWR?" H 4850 4200 50  0001 C CNN
+F 0 "#PWR026" H 4850 4200 50  0001 C CNN
 F 1 "+3V3" H 4865 4523 50  0000 C CNN
 F 2 "" H 4850 4350 50  0001 C CNN
@@
 	2600 5250 4850 5250
 $Comp
-L AVR-KiCAD-Lib-Resistors:RC0402FR-071KL R?
+L AVR-KiCAD-Lib-Resistors:RC0402FR-071KL R9
 U 1 1 5F00F6CF
 P 4550 4550
-F 0 "R?" V 4504 4637 50  0000 L CNN
+F 0 "R9" V 4504 4637 50  0000 L CNN
 F 1 "RC0402FR-071KL" V 4550 4638 50  0001 L CNN
 F 2 "AVR-KiCAD-Lib-Resistors:R0402" H 4550 4550 50  0001 C CNN
@@
 RS485_SL_RATE2
 $Comp
-L AVR-KiCAD-Lib-Resistors:RC0402FR-071KL R?
+L AVR-KiCAD-Lib-Resistors:RC0402FR-071KL R7
 U 1 1 5F01A8A5
 P 2600 5650
-F 0 "R?" V 2554 5737 50  0000 L CNN
+F 0 "R7" V 2554 5737 50  0000 L CNN
 F 1 "RC0402FR-071KL" V 2600 5738 50  0001 L CNN
 F 2 "AVR-KiCAD-Lib-Resistors:R0402" H 2600 5650 50  0001 C CNN
@@
 	4850 5450 2600 5450
 $Comp
-L power:GND #PWR?
+L power:GND #PWR015
 U 1 1 5F022281
 P 2600 5850
-F 0 "#PWR?" H 2600 5600 50  0001 C CNN
+F 0 "#PWR015" H 2600 5600 50  0001 C CNN
 F 1 "GND" H 2605 5677 50  0000 C CNN
 F 2 "" H 2600 5850 50  0001 C CNN
@@
 $EndComp
 $Comp
-L AVR-KiCAD-Lib-Resistors:RC0402FR-071KL R?
+L AVR-KiCAD-Lib-Resistors:RC0402FR-071KL R6
 U 1 1 5F027579
 P 2600 2450
-F 0 "R?" V 2554 2537 50  0000 L CNN
+F 0 "R6" V 2554 2537 50  0000 L CNN
 F 1 "RC0402FR-071KL" V 2600 2538 50  0001 L CNN
 F 2 "AVR-KiCAD-Lib-Resistors:R0402" H 2600 2450 50  0001 C CNN
@@
 	4850 2250 2600 2250
 $Comp
-L power:GND #PWR?
+L power:GND #PWR014
 U 1 1 5F027580
 P 2600 2650
-F 0 "#PWR?" H 2600 2400 50  0001 C CNN
+F 0 "#PWR014" H 2600 2400 50  0001 C CNN
 F 1 "GND" H 2605 2477 50  0000 C CNN
 F 2 "" H 2600 2650 50  0001 C CNN
@@
 RS485_SL_RATE1
 $Comp
-L AVR-KiCAD-Lib-Resistors:RC0402FR-071KL R?
+L AVR-KiCAD-Lib-Resistors:RC0402FR-071KL R8
 U 1 1 5F044D3C
 P 4550 1350
-F 0 "R?" V 4504 1437 50  0000 L CNN
+F 0 "R8" V 4504 1437 50  0000 L CNN
 F 1 "RC0402FR-071KL" V 4550 1438 50  0001 L CNN
 F 2 "AVR-KiCAD-Lib-Resistors:R0402" H 4550 1350 50  0001 C CNN
@@
 RS485_TERM_EN2
 $Comp
-L power:GND #PWR?
+L power:GND #PWR018
 U 1 1 5F017F66
 P 3350 3500
-F 0 "#PWR?" H 3350 3250 50  0001 C CNN
+F 0 "#PWR018" H 3350 3250 50  0001 C CNN
 F 1 "GND" H 3355 3327 50  0000 C CNN
 F 2 "" H 3350 3500 50  0001 C CNN
@@
 $EndComp
 $Comp
-L power:+3V3 #PWR?
+L power:+3V3 #PWR017
 U 1 1 5F0382CD
 P 2950 6150
-F 0 "#PWR?" H 2950 6000 50  0001 C CNN
+F 0 "#PWR017" H 2950 6000 50  0001 C CNN
 F 1 "+3V3" H 2965 6323 50  0000 C CNN
 F 2 "" H 2950 6150 50  0001 C CNN
