File: PCB/Cape/agricoltura-madre-cape-B/agricoltura-madre-cape-B.kicad_pcb (KiCad board)
At the start: 2 copper layers, 54.6 x 86.4 mm, 2 parts, among them P8 BeagleBone_Black_Header, P9 BeagleBone_Black_Header

Commit message: KiCAD 8
Projected updated to KiCAD 8
Other:
- outline, holes or cut-outs redrawn
- net class Default removed
